Commit message: integrate redundancy resolution plugin

File: coordinated_motion_examples/urdf/robot6R_macro.xacro (robot description, xacro)
@@ -100,5 +100,5 @@
         <origin xyz="0 0 0" rpy="${pi / 2.0} 0 0" />
         <geometry>
-                <cylinder length="${joint_length}" radius="${joint_radius}"/>
+          <cylinder length="${joint_length}" radius="${joint_radius}"/>
         </geometry>
         <material name="grey"/>
@@ -107,5 +107,5 @@
         <origin xyz="0 ${link4_length / 2.0} 0" rpy="${pi / 2.0} 0 0" />
         <geometry>
-                <cylinder length="${link4_length}" radius="${link_radius}"/>
+          <cylinder length="${link4_length}" radius="${link_radius}"/>
         </geometry>
         <material name="grey"/>
@@ -114,5 +114,5 @@
         <origin xyz="0 ${link4_length} 0" rpy="0 0 0" />
         <geometry>
-                <cylinder length="${joint_length}" radius="${joint_radius}"/>
+          <cylinder length="${joint_length}" radius="${joint_radius}"/>
         </geometry>
         <material name="grey"/>
@@ -216,4 +216,10 @@
       </visual>
     </link>
+    <link name="${prefix}tool"/>
+    <joint name="${prefix}tool_joint" type="fixed">
+      <origin xyz="0 0 0" rpy="${-pi/2} ${-pi/2} 0"/>
+      <parent link="${prefix}tool0"/>
+      <child link="${prefix}tool"/>
+    </joint>
   </xacro:macro>
 </robot>
