Commit message: WIP: migrate coordinated_motion_examples

File: coordinated_motion_examples/urdf/two_robot6R.xacro (robot description, xacro)
@@ -6,7 +6,7 @@
   <xacro:robot6R_macro prefix="rob1_"/>
   <xacro:robot6R_macro prefix="rob2_"/>
-  <xacro:include filename="$(find coordinated_motion_examples)/urdf/positioner1R_macro.xacro"/>
-  <xacro:positioner1R_macro/>
-  <!-- colors -->
+  <!-- <xacro:include filename="$(find coordinated_motion_examples)/urdf/positioner1R_macro.xacro"/> -->
+  <!-- <xacro:positioner1R_macro/> -->
+  <!-- Colors -->
   <material name="grey">
     <color rgba="0.7 0.7 0.7 1.0"/>
@@ -24,9 +24,13 @@
     <origin xyz="${radius} ${spacing/2} 0.0" rpy="0.0 0.0 ${pi}"/>
   </joint>
-  <joint name="positioner_joint" type="continuous">
-    <parent link="world"/>
-    <child link = "positioner_base"/>
-    <origin xyz="0.0 0.0 0.0" rpy="0.0 0.0 0.0"/>
-    <axis xyz="0 0 1"/>
-  </joint>
+  <!-- <joint name="positioner_joint" type="continuous"> -->
+  <!--   <parent link="world"/> -->
+  <!--   <child link = "positioner_base"/> -->
+  <!--   <origin xyz="0.0 0.0 0.0" rpy="0.0 0.0 0.0"/> -->
+  <!--   <axis xyz="0 0 1"/> -->
+  <!-- </joint> -->
+  <!-- ROS2 control -->
+  <xacro:include filename="$(find taskspace_control_examples)/urdf/robot6R.ros2_control.xacro"/>
+  <xacro:robot6R_ros2_control prefix="rob1_"/>
+  <xacro:robot6R_ros2_control prefix="rob2_"/>
 </robot>

Commit message: WIP: add positioner controller

File: coordinated_motion_examples/urdf/two_robot6R.xacro (robot description, xacro)
@@ -6,6 +6,6 @@
   <xacro:robot6R_macro prefix="rob1_"/>
   <xacro:robot6R_macro prefix="rob2_"/>
-  <!-- <xacro:include filename="$(find coordinated_motion_examples)/urdf/positioner1R_macro.xacro"/> -->
-  <!-- <xacro:positioner1R_macro/> -->
+  <xacro:include filename="$(find coordinated_motion_examples)/urdf/positioner1R_macro.xacro"/>
+  <xacro:positioner1R_macro/>
   <!-- Colors -->
   <material name="grey">
@@ -24,13 +24,15 @@
     <origin xyz="${radius} ${spacing/2} 0.0" rpy="0.0 0.0 ${pi}"/>
   </joint>
-  <!-- <joint name="positioner_joint" type="continuous"> -->
-  <!--   <parent link="world"/> -->
-  <!--   <child link = "positioner_base"/> -->
-  <!--   <origin xyz="0.0 0.0 0.0" rpy="0.0 0.0 0.0"/> -->
-  <!--   <axis xyz="0 0 1"/> -->
-  <!-- </joint> -->
+  <joint name="positioner_joint" type="continuous">
+    <parent link="world"/>
+    <child link = "positioner_base"/>
+    <origin xyz="0.0 0.0 0.0" rpy="0.0 0.0 0.0"/>
+    <axis xyz="0 0 1"/>
+  </joint>
   <!-- ROS2 control -->
   <xacro:include filename="$(find taskspace_control_examples)/urdf/robot6R.ros2_control.xacro"/>
   <xacro:robot6R_ros2_control prefix="rob1_"/>
   <xacro:robot6R_ros2_control prefix="rob2_"/>
+  <xacro:include filename="$(find coordinated_motion_examples)/urdf/positioner1R.ros2_control.xacro"/>
+  <xacro:positioner_ros2_control prefix=""/>
 </robot>
