Commit message: implement positioner state interfaces
Two interfaces are provided. A `loaned` interface and a `topic`
interface.

- `loaned`: Uses a reference to the ros2_control state interface
- `topic`: Subscribes to the joint state of the positioner

File: coordinated_motion_examples/urdf/positioner1R.ros2_control.xacro (robot description, xacro)
@@ -2,16 +2,11 @@
 <robot xmlns:xacro="http://www.ros.org/wiki/xacro">
   <xacro:macro name="positioner_ros2_control" params="prefix">
-    <ros2_control name="${prefix}ros2_control" type="system">
-      <hardware>
-        <plugin>mock_components/GenericSystem</plugin>
-      </hardware>
-      <joint name="${prefix}positioner_joint">
-        <command_interface name="position"/>
-        <state_interface name="position">
-          <param name="initial_value">0.0</param>
-        </state_interface>
-        <state_interface name="velocity"/>
-      </joint>
-    </ros2_control>
+    <joint name="${prefix}positioner_joint">
+      <command_interface name="position"/>
+      <state_interface name="position">
+        <param name="initial_value">0.0</param>
+      </state_interface>
+      <state_interface name="velocity"/>
+    </joint>
   </xacro:macro>
 </robot>

File: coordinated_motion_examples/urdf/two_robot6R.xacro (robot description, xacro)
@@ -1,4 +1,4 @@
 <?xml version="1.0"?>
-<robot name="two_robot6R" xmlns:xacro="http://ros.org/wiki/xacro">
+<robot name="two_robot6R" xmlns:xacro="http://www.ros.org/wiki/xacro">
   <xacro:property name="radius" value="0.5"/>
   <xacro:property name="spacing" value="0.52"/>
@@ -31,8 +31,13 @@
   </joint>
   <!-- ROS2 control -->
-  <xacro:include filename="$(find taskspace_control_examples)/urdf/robot6R.ros2_control.xacro"/>
-  <xacro:robot6R_ros2_control prefix="rob1_"/>
-  <xacro:robot6R_ros2_control prefix="rob2_"/>
+  <xacro:include filename="$(find coordinated_motion_examples)/urdf/robot6R.ros2_control.xacro"/>
   <xacro:include filename="$(find coordinated_motion_examples)/urdf/positioner1R.ros2_control.xacro"/>
-  <xacro:positioner_ros2_control prefix=""/>
+  <ros2_control name="two_robot_ros2_control" type="system">
+    <hardware>
+      <plugin>mock_components/GenericSystem</plugin>
+    </hardware>
+    <xacro:robot6R_ros2_control prefix="rob1_"/>
+    <xacro:robot6R_ros2_control prefix="rob2_"/>
+    <xacro:positioner_ros2_control prefix=""/>
+  </ros2_control>
 </robot>

File: coordinated_motion_examples/urdf/two_robot7R.xacro (robot description, xacro)
@@ -34,8 +34,13 @@
   </joint>
   <!-- ROS2 control -->
-  <xacro:include filename="$(find taskspace_control_examples)/urdf/robot7R.ros2_control.xacro"/>
-  <xacro:robot7R_ros2_control prefix="rob1_"/>
-  <xacro:robot7R_ros2_control prefix="rob2_"/>
+  <xacro:include filename="$(find coordinated_motion_examples)/urdf/robot7R.ros2_control.xacro"/>
   <xacro:include filename="$(find coordinated_motion_examples)/urdf/positioner1R.ros2_control.xacro"/>
-  <xacro:positioner_ros2_control prefix=""/>
+  <ros2_control name="two_robot_ros2_control" type="system">
+    <hardware>
+      <plugin>mock_components/GenericSystem</plugin>
+    </hardware>
+    <xacro:robot7R_ros2_control prefix="rob1_"/>
+    <xacro:robot7R_ros2_control prefix="rob2_"/>
+    <xacro:positioner_ros2_control prefix=""/>
+  </ros2_control>
 </robot>
